Commit message: 增加底盘建图功能程序

File: tracer_description/urdf/tracer_v1.xacro (robot description, xacro)
@@ -33,4 +33,10 @@
     <xacro:property name="wheel_length" value="0.8e-01" />
     <xacro:property name="wheel_radius" value="1.600e-01" />
+    <link name="base_footprint" />
+    <joint name="base_footprint_base_link" type="fixed">
+        <origin xyz="0 0 0.15" rpy="0 0 0" />
+        <parent link="base_footprint" />
+        <child link="base_link" />
+    </joint>
     <!-- Base link -->
     <link name="base_link">
