Commit message: 优化MC+小车模型整体拼接

File: myarm_description/urdf/myarm_c650/myarm_c650.urdf (robot description, URDF)
Before this commit: robot firefighter, 9 links, 8 joints
Links:
- link base: geometry collision mesh filename=package://mycobot_description/urdf/myarm_c650/myarm_basic_b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; visual mesh filename=package://mycobot_description/urdf/myarm_c650/myarm_basic_b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
- link gripper: geometry collision mesh filename=package://mycobot_description/urdf/myarm_c650/myarm_c_grip_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; visual mesh filename=package://mycobot_description/urdf/myarm_c650/myarm_c_grip_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
- link gripper_left: geometry collision mesh filename=package://mycobot_description/urdf/myarm_c650/myarm_c_grip_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; visual mesh filename=package://mycobot_description/urdf/myarm_c650/myarm_c_grip_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
- link gripper_right: geometry collision mesh filename=package://mycobot_description/urdf/myarm_c650/myarm_c_grip_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; visual mesh filename=package://mycobot_description/urdf/myarm_c650/myarm_c_grip_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
- link link1: geometry collision mesh filename=package://mycobot_description/urdf/myarm_c650/joint1.dae; visual mesh filename=package://mycobot_description/urdf/myarm_c650/joint1.dae
- link link2: geometry collision mesh filename=package://mycobot_description/urdf/myarm_c650/joint2.dae; visual mesh filename=package://mycobot_description/urdf/myarm_c650/joint2.dae
- link link3: geometry collision mesh filename=package://mycobot_description/urdf/myarm_c650/joint3.dae; visual mesh filename=package://mycobot_description/urdf/myarm_c650/joint3.dae
- link link4: geometry collision mesh filename=package://mycobot_description/urdf/myarm_c650/joint4.dae; visual mesh filename=package://mycobot_description/urdf/myarm_c650/joint4.dae
- link link5: geometry collision mesh filename=package://mycobot_description/urdf/myarm_c650/joint5.dae; visual mesh filename=package://mycobot_description/urdf/myarm_c650/joint5.dae
Joints:
- joint joint1: axis 0 0 1 -> 0 0 -1
- joint joint4: axis  0 0 1 ->  0 0 -1
- joint joint6: axis 0 0 1 -> 0 0 -1

File: myarm_description/urdf/myarm_m/myarm_m.urdf (robot description, URDF)
Before this commit: robot myarm_m, 9 links, 8 joints
Joints:
- joint joint1: axis 0 0 1 -> 0 0 -1
- joint joint2: axis 0 0 1 -> 0 0 -1
- joint joint3: axis  0 0 1 ->  0 0 -1; limit lower=-1.5882 upper=1.7977 effort=1000.0 velocity=0 -> lower=-1.5882 upper=1.2977 effort=1000.0 velocity=0
- joint joint4: axis  0 0 1 ->  0 0 -1
- joint joint6: axis 0 0 1 -> 0 0 -1
