Commit message: 增加MC手臂联调控制脚本

File: myarm_description/urdf/myarm_c650/myarm_c1.xacro (robot description, xacro)
@@ -5,5 +5,5 @@
     <visual>
       <geometry>
-       <mesh filename="package://mycobot_description/urdf/myarm_c650/myarm_basic_base.dae"/>
+       <mesh filename="package://myarm_description/urdf/myarm_c650/myarm_basic_base.dae"/>
       </geometry>
       <origin xyz = "0.0 0 0 " rpy = " 0 0 0"/>
@@ -11,5 +11,5 @@
     <collision>
       <geometry>
-       <mesh filename="package://mycobot_description/urdf/myarm_c650/myarm_basic_base.dae"/>
+       <mesh filename="package://myarm_description/urdf/myarm_c650/myarm_basic_base.dae"/>
         </geometry>
         <origin xyz = "0.0 0 0 " rpy = " 0 0 0"/>
@@ -19,5 +19,5 @@
     <visual>
       <geometry>
-       <mesh filename="package://mycobot_description/urdf/myarm_c650/joint1.dae"/>
+       <mesh filename="package://myarm_description/urdf/myarm_c650/joint1.dae"/>
       </geometry>
       <origin xyz = "0.0 0 0.0065 " rpy = " 3.14159 0 0"/>
@@ -25,5 +25,5 @@
     <collision>
      <geometry>
-       <mesh filename="package://mycobot_description/urdf/myarm_c650/joint1.dae"/>
+       <mesh filename="package://myarm_description/urdf/myarm_c650/joint1.dae"/>
       </geometry>
       <origin xyz = "0.0 0 0.0065 " rpy = " 3.14159 0 0"/>
@@ -33,5 +33,5 @@
     <visual>
       <geometry>
-       <mesh filename="package://mycobot_description/urdf/myarm_c650/joint2.dae"/>
+       <mesh filename="package://myarm_description/urdf/myarm_c650/joint2.dae"/>
       </geometry>
     <origin xyz = "0.0 0.003 0.0 " rpy = " 3.14159 0 -1.5708 "/>
@@ -39,5 +39,5 @@
     <collision>
       <geometry>
-       <mesh filename="package://mycobot_description/urdf/myarm_c650/joint2.dae"/>
+       <mesh filename="package://myarm_description/urdf/myarm_c650/joint2.dae"/>
       </geometry>
       <origin xyz = "0.0 0.003 0.0 " rpy = " 3.14159 0 -1.5708"/>
@@ -47,5 +47,5 @@
     <visual>
       <geometry>
-       <mesh filename="package://mycobot_description/urdf/myarm_c650/joint3.dae"/>
+       <mesh filename="package://myarm_description/urdf/myarm_c650/joint3.dae"/>
       </geometry>
       <origin xyz = "0.0 -0.001 0.004 " rpy = " 0 0 0"/>
@@ -53,5 +53,5 @@
     <collision>
       <geometry>
-       <mesh filename="package://mycobot_description/urdf/myarm_c650/joint3.dae"/>
+       <mesh filename="package://myarm_description/urdf/myarm_c650/joint3.dae"/>
       </geometry>
       <origin xyz = "0.0 -0.001 0.004" rpy = " 0 0 0"/>
@@ -61,5 +61,5 @@
     <visual>
       <geometry>
-       <mesh filename="package://mycobot_description/urdf/myarm_c650/joint4.dae"/>
+       <mesh filename="package://myarm_description/urdf/myarm_c650/joint4.dae"/>
       </geometry>
     <origin xyz = "0.0 0 0.004 " rpy = " 0 3.14159 0"/>
@@ -67,5 +67,5 @@
     <collision>
        <geometry>
-       <mesh filename="package://mycobot_description/urdf/myarm_c650/joint4.dae"/>
+       <mesh filename="package://myarm_description/urdf/myarm_c650/joint4.dae"/>
       </geometry>
       <origin xyz = "0.0 0 0.004 " rpy = " 0 3.14159 0"/>
@@ -75,5 +75,5 @@
     <visual>
       <geometry>
-       <mesh filename="package://mycobot_description/urdf/myarm_c650/joint5.dae"/>
+       <mesh filename="package://myarm_description/urdf/myarm_c650/joint5.dae"/>
       </geometry>
     <origin xyz = "0 0.009 0.001 " rpy = " 3.14159 0 -1.5708"/>
@@ -81,5 +81,5 @@
     <collision>
       <geometry>
-       <mesh filename="package://mycobot_description/urdf/myarm_c650/joint5.dae"/>
+       <mesh filename="package://myarm_description/urdf/myarm_c650/joint5.dae"/>
       </geometry>
     <origin xyz = "0 0.009 0.001 " rpy = " 3.14159 0 -1.5708"/>
@@ -89,5 +89,5 @@
     <visual>
       <geometry>
-       <mesh filename="package://mycobot_description/urdf/myarm_c650/myarm_c_grip_Base.dae"/>
+       <mesh filename="package://myarm_description/urdf/myarm_c650/myarm_c_grip_Base.dae"/>
       </geometry>
     <origin xyz = "0 0 0.003 " rpy = " 3.14159 0 0"/>
@@ -95,5 +95,5 @@
     <collision>
       <geometry>
-       <mesh filename="package://mycobot_description/urdf/myarm_c650/myarm_c_grip_Base.dae"/>
+       <mesh filename="package://myarm_description/urdf/myarm_c650/myarm_c_grip_Base.dae"/>
       </geometry>
     <origin xyz = "0 0 0.003 " rpy = " 3.14159 0 0"/>
@@ -103,5 +103,5 @@
     <visual>
       <geometry>
-       <mesh filename="package://mycobot_description/urdf/myarm_c650/myarm_c_grip_R.dae"/>
+       <mesh filename="package://myarm_description/urdf/myarm_c650/myarm_c_grip_R.dae"/>
       </geometry>
     <origin xyz = "0.010 0 0 " rpy = " 1.5708 3.14159 -1.5708"/>
@@ -109,5 +109,5 @@
     <collision>
       <geometry>
-       <mesh filename="package://mycobot_description/urdf/myarm_c650/myarm_c_grip_R.dae"/>
+       <mesh filename="package://myarm_description/urdf/myarm_c650/myarm_c_grip_R.dae"/>
       </geometry>
     <origin xyz = "0.010 0 0 " rpy = " 1.5708 3.14159 -1.5708"/>
@@ -117,5 +117,5 @@
     <visual>
       <geometry>
-       <mesh filename="package://mycobot_description/urdf/myarm_c650/myarm_c_grip_L.dae"/>
+       <mesh filename="package://myarm_description/urdf/myarm_c650/myarm_c_grip_L.dae"/>
       </geometry>
     <origin xyz = "0.010 0 0 " rpy = " 1.5708 3.14159 -1.5708"/>
@@ -123,5 +123,5 @@
     <collision>
       <geometry>
-       <mesh filename="package://mycobot_description/urdf/myarm_c650/myarm_c_grip_L.dae"/>
+       <mesh filename="package://myarm_description/urdf/myarm_c650/myarm_c_grip_L.dae"/>
       </geometry>
     <origin xyz = "0.010 0 0 " rpy = " 1.5708 3.14159 -1.5708"/>

File: myarm_description/urdf/myarm_c650/myarm_c2.xacro (robot description, xacro)
@@ -5,5 +5,5 @@
     <visual>
       <geometry>
-       <mesh filename="package://mycobot_description/urdf/myarm_c650/myarm_basic_base.dae"/>
+       <mesh filename="package://myarm_description/urdf/myarm_c650/myarm_basic_base.dae"/>
       </geometry>
       <origin xyz = "0.0 0 0 " rpy = " 0 0 0"/>
@@ -11,5 +11,5 @@
     <collision>
       <geometry>
-       <mesh filename="package://mycobot_description/urdf/myarm_c650/myarm_basic_base.dae"/>
+       <mesh filename="package://myarm_description/urdf/myarm_c650/myarm_basic_base.dae"/>
         </geometry>
         <origin xyz = "0.0 0 0 " rpy = " 0 0 0"/>
@@ -19,5 +19,5 @@
     <visual>
       <geometry>
-       <mesh filename="package://mycobot_description/urdf/myarm_c650/joint1.dae"/>
+       <mesh filename="package://myarm_description/urdf/myarm_c650/joint1.dae"/>
       </geometry>
       <origin xyz = "0.0 0 0.0065 " rpy = " 3.14159 0 0"/>
@@ -25,5 +25,5 @@
     <collision>
      <geometry>
-       <mesh filename="package://mycobot_description/urdf/myarm_c650/joint1.dae"/>
+       <mesh filename="package://myarm_description/urdf/myarm_c650/joint1.dae"/>
       </geometry>
       <origin xyz = "0.0 0 0.0065 " rpy = " 3.14159 0 0"/>
@@ -33,5 +33,5 @@
     <visual>
       <geometry>
-       <mesh filename="package://mycobot_description/urdf/myarm_c650/joint2.dae"/>
+       <mesh filename="package://myarm_description/urdf/myarm_c650/joint2.dae"/>
       </geometry>
     <origin xyz = "0.0 0.003 0.0 " rpy = " 3.14159 0 -1.5708 "/>
@@ -39,5 +39,5 @@
     <collision>
       <geometry>
-       <mesh filename="package://mycobot_description/urdf/myarm_c650/joint2.dae"/>
+       <mesh filename="package://myarm_description/urdf/myarm_c650/joint2.dae"/>
       </geometry>
       <origin xyz = "0.0 0.003 0.0 " rpy = " 3.14159 0 -1.5708"/>
@@ -47,5 +47,5 @@
     <visual>
       <geometry>
-       <mesh filename="package://mycobot_description/urdf/myarm_c650/joint3.dae"/>
+       <mesh filename="package://myarm_description/urdf/myarm_c650/joint3.dae"/>
       </geometry>
       <origin xyz = "0.0 -0.001 0.004 " rpy = " 0 0 0"/>
@@ -53,5 +53,5 @@
     <collision>
       <geometry>
-       <mesh filename="package://mycobot_description/urdf/myarm_c650/joint3.dae"/>
+       <mesh filename="package://myarm_description/urdf/myarm_c650/joint3.dae"/>
       </geometry>
       <origin xyz = "0.0 -0.001 0.004" rpy = " 0 0 0"/>
@@ -61,5 +61,5 @@
     <visual>
       <geometry>
-       <mesh filename="package://mycobot_description/urdf/myarm_c650/joint4.dae"/>
+       <mesh filename="package://myarm_description/urdf/myarm_c650/joint4.dae"/>
       </geometry>
     <origin xyz = "0.0 0 0.004 " rpy = " 0 3.14159 0"/>
@@ -67,5 +67,5 @@
     <collision>
        <geometry>
-       <mesh filename="package://mycobot_description/urdf/myarm_c650/joint4.dae"/>
+       <mesh filename="package://myarm_description/urdf/myarm_c650/joint4.dae"/>
       </geometry>
       <origin xyz = "0.0 0 0.004 " rpy = " 0 3.14159 0"/>
@@ -75,5 +75,5 @@
     <visual>
       <geometry>
-       <mesh filename="package://mycobot_description/urdf/myarm_c650/joint5.dae"/>
+       <mesh filename="package://myarm_description/urdf/myarm_c650/joint5.dae"/>
       </geometry>
     <origin xyz = "0 0.009 0.001 " rpy = " 3.14159 0 -1.5708"/>
@@ -81,5 +81,5 @@
     <collision>
       <geometry>
-       <mesh filename="package://mycobot_description/urdf/myarm_c650/joint5.dae"/>
+       <mesh filename="package://myarm_description/urdf/myarm_c650/joint5.dae"/>
       </geometry>
     <origin xyz = "0 0.009 0.001 " rpy = " 3.14159 0 -1.5708"/>
@@ -89,5 +89,5 @@
     <visual>
       <geometry>
-       <mesh filename="package://mycobot_description/urdf/myarm_c650/myarm_c_grip_Base.dae"/>
+       <mesh filename="package://myarm_description/urdf/myarm_c650/myarm_c_grip_Base.dae"/>
       </geometry>
     <origin xyz = "0 0 0.003 " rpy = " 3.14159 0 0"/>
@@ -95,5 +95,5 @@
     <collision>
       <geometry>
-       <mesh filename="package://mycobot_description/urdf/myarm_c650/myarm_c_grip_Base.dae"/>
+       <mesh filename="package://myarm_description/urdf/myarm_c650/myarm_c_grip_Base.dae"/>
       </geometry>
     <origin xyz = "0 0 0.003 " rpy = " 3.14159 0 0"/>
@@ -103,5 +103,5 @@
     <visual>
       <geometry>
-       <mesh filename="package://mycobot_description/urdf/myarm_c650/myarm_c_grip_R.dae"/>
+       <mesh filename="package://myarm_description/urdf/myarm_c650/myarm_c_grip_R.dae"/>
       </geometry>
     <origin xyz = "0.010 0 0 " rpy = " 1.5708 3.14159 -1.5708"/>
@@ -109,5 +109,5 @@
     <collision>
       <geometry>
-       <mesh filename="package://mycobot_description/urdf/myarm_c650/myarm_c_grip_R.dae"/>
+       <mesh filename="package://myarm_description/urdf/myarm_c650/myarm_c_grip_R.dae"/>
       </geometry>
     <origin xyz = "0.010 0 0 " rpy = " 1.5708 3.14159 -1.5708"/>
@@ -117,5 +117,5 @@
     <visual>
       <geometry>
-       <mesh filename="package://mycobot_description/urdf/myarm_c650/myarm_c_grip_L.dae"/>
+       <mesh filename="package://myarm_description/urdf/myarm_c650/myarm_c_grip_L.dae"/>
       </geometry>
     <origin xyz = "0.010 0 0 " rpy = " 1.5708 3.14159 -1.5708"/>
@@ -123,5 +123,5 @@
     <collision>
       <geometry>
-       <mesh filename="package://mycobot_description/urdf/myarm_c650/myarm_c_grip_L.dae"/>
+       <mesh filename="package://myarm_description/urdf/myarm_c650/myarm_c_grip_L.dae"/>
       </geometry>
     <origin xyz = "0.010 0 0 " rpy = " 1.5708 3.14159 -1.5708"/>

File: myarm_description/urdf/myarm_c650/myarm_c650.urdf (robot description, URDF)
Before this commit: robot firefighter, 9 links, 8 joints
Links:
- link base: geometry collision mesh filename=package://myarm_description/urdf/myarm_c650/myarm_basic_bas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; visual mesh filename=package://myarm_description/urdf/myarm_c650/myarm_basic_bas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
- link gripper: geometry collision mesh filename=package://myarm_description/urdf/myarm_c650/myarm_c_grip_Ba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; visual mesh filename=package://myarm_description/urdf/myarm_c650/myarm_c_grip_Ba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
- link gripper_left: geometry collision mesh filename=package://myarm_description/urdf/myarm_c650/myarm_c_grip_R.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; visual mesh filename=package://myarm_description/urdf/myarm_c650/myarm_c_grip_R.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
- link gripper_right: geometry collision mesh filename=package://myarm_description/urdf/myarm_c650/myarm_c_grip_L.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; visual mesh filename=package://myarm_description/urdf/myarm_c650/myarm_c_grip_L.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
- link link1: geometry collision mesh filename=package://myarm_description/urdf/myarm_c650/joint1.dae; visual mesh filename=package://myarm_description/urdf/myarm_c650/joint1.dae
- link link2: geometry collision mesh filename=package://myarm_description/urdf/myarm_c650/joint2.dae; visual mesh filename=package://myarm_description/urdf/myarm_c650/joint2.dae
- link link3: geometry collision mesh filename=package://myarm_description/urdf/myarm_c650/joint3.dae; visual mesh filename=package://myarm_description/urdf/myarm_c650/joint3.dae
- link link4: geometry collision mesh filename=package://myarm_description/urdf/myarm_c650/joint4.dae; visual mesh filename=package://myarm_description/urdf/myarm_c650/joint4.dae
- link link5: geometry collision mesh filename=package://myarm_description/urdf/myarm_c650/joint5.dae; visual mesh filename=package://myarm_description/urdf/myarm_c650/joint5.dae
