Commit message: 更新模型运动方向

File: myarm_description/urdf/myarm_m/myarm_m1.xacro (robot description, xacro)
@@ -143,5 +143,5 @@
 </joint>
  <joint name="m1_joint3" type="revolute">
-  <axis xyz=" 0 0 -1"/>
+  <axis xyz=" 0 0 1"/>
   <limit effort = "1000.0" lower = "-1.5882" upper = "1.7977" velocity = "0"/>
   <parent link="m1_link2"/>

File: myarm_description/urdf/myarm_m/myarm_m2.xacro (robot description, xacro)
@@ -143,5 +143,5 @@
 </joint>
  <joint name="m2_joint3" type="revolute">
-  <axis xyz=" 0 0 -1"/>
+  <axis xyz=" 0 0 1"/>
   <limit effort = "1000.0" lower = "-1.5882" upper = "1.7977" velocity = "0"/>
   <parent link="m2_link2"/>

Commit message: update arm control code

File: myarm_description/urdf/myarm_m/myarm_m1.xacro (robot description, xacro)
@@ -143,5 +143,5 @@
 </joint>
  <joint name="m1_joint3" type="revolute">
-  <axis xyz=" 0 0 1"/>
+  <axis xyz=" 0 0 -1"/>
   <limit effort = "1000.0" lower = "-1.5882" upper = "1.7977" velocity = "0"/>
   <parent link="m1_link2"/>

File: myarm_description/urdf/myarm_m/myarm_m2.xacro (robot description, xacro)
@@ -143,5 +143,5 @@
 </joint>
  <joint name="m2_joint3" type="revolute">
-  <axis xyz=" 0 0 1"/>
+  <axis xyz=" 0 0 -1"/>
   <limit effort = "1000.0" lower = "-1.5882" upper = "1.7977" velocity = "0"/>
   <parent link="m2_link2"/>
