Commit message: update ranger mini3.0 corde

File: ranger_mini_v3/urdf/ranger_mini.xacro (robot description, xacro)
@@ -3,5 +3,5 @@
   <link name="base_footprint" />
     <joint name="base_footprint_base_link" type="fixed">
-        <origin xyz="0 0 0.15" rpy="0 0 0" />
+        <origin xyz="0 0 0.32" rpy="0 0 0" />
         <parent link="base_footprint" />
         <child link="base_link" />
